File: A1200-adapter/A1200-adapter.kicad_pcb (KiCad board)
At the start: 2 copper layers, 26.1 x 139 mm, 2 parts, among them CON1 A3000_A4000_LOCAL_BUS_SLOT, CON2 A1200-EXP

Commit message: Add files via upload
Connections:
- CON1 pad 1: Net-(CON1-Pad1) -> /DSACK1
- CON1 pad 10: Net-(CON1-Pad10) -> GND
- CON1 pad 100: Net-(CON1-Pad100) -> /ECS
- CON1 pad 102: Net-(CON1-Pad102) -> +5V
- CON1 pad 103: Net-(CON1-Pad103) -> +5V
- CON1 pad 105: Net-(CON1-Pad105) -> /BG
- CON1 pad 106: Net-(CON1-Pad106) -> +5V
- CON1 pad 107: Net-(CON1-Pad107) -> +5V
- CON1 pad 108: Net-(CON1-Pad108) -> /RMC
- CON1 pad 109: Net-(CON1-Pad109) -> /RST
- CON1 pad 11: Net-(CON1-Pad11) -> GND
- CON1 pad 115: Net-(CON1-Pad115) -> GND
- CON1 pad 117: Net-(CON1-Pad117) -> /RESET
- CON1 pad 118: Net-(CON1-Pad118) -> GND
- CON1 pad 119: Net-(CON1-Pad119) -> GND
- CON1 pad 12: Net-(CON1-Pad12) -> /AVEC
- CON1 pad 120: Net-(CON1-Pad120) -> /IPL0
- CON1 pad 121: Net-(CON1-Pad121) -> /SIZ0
- CON1 pad 124: Net-(CON1-Pad124) -> /IPL1
- CON1 pad 125: Net-(CON1-Pad125) -> /FC2
- CON1 pad 127: Net-(CON1-Pad127) -> GND
- CON1 pad 128: Net-(CON1-Pad128) -> /IPL2
- CON1 pad 129: Net-(CON1-Pad129) -> /SIZ1
- CON1 pad 130: Net-(CON1-Pad130) -> GND
- CON1 pad 131: Net-(CON1-Pad131) -> GND
- CON1 pad 133: Net-(CON1-Pad133) -> /AS
- CON1 pad 134: Net-(CON1-Pad134) -> /FPUCS
- CON1 pad 135: Net-(CON1-Pad135) -> /CPUCLK
- CON1 pad 136: Net-(CON1-Pad136) -> /OCS
- CON1 pad 137: Net-(CON1-Pad137) -> /D31
- CON1 pad 138: Net-(CON1-Pad138) -> GND
- CON1 pad 139: Net-(CON1-Pad139) -> GND
- CON1 pad 14: Net-(CON1-Pad14) -> +5V
- CON1 pad 140: Net-(CON1-Pad140) -> /D15
- CON1 pad 141: Net-(CON1-Pad141) -> /D30
- CON1 pad 142: Net-(CON1-Pad142) -> GND
- CON1 pad 143: Net-(CON1-Pad143) -> GND
- CON1 pad 144: Net-(CON1-Pad144) -> /D14
- CON1 pad 145: Net-(CON1-Pad145) -> /D29
- CON1 pad 148: Net-(CON1-Pad148) -> /D13
- CON1 pad 149: Net-(CON1-Pad149) -> /D28
- CON1 pad 15: Net-(CON1-Pad15) -> +5V
- CON1 pad 151: Net-(CON1-Pad151) -> GND
- CON1 pad 152: Net-(CON1-Pad152) -> /D12
- CON1 pad 153: Net-(CON1-Pad153) -> /D27
- CON1 pad 154: Net-(CON1-Pad154) -> GND
- CON1 pad 155: Net-(CON1-Pad155) -> GND
- CON1 pad 156: Net-(CON1-Pad156) -> /D11
- CON1 pad 157: Net-(CON1-Pad157) -> /D26
- CON1 pad 160: Net-(CON1-Pad160) -> /D10
- CON1 pad 161: Net-(CON1-Pad161) -> /D25
- CON1 pad 163: Net-(CON1-Pad163) -> GND
- CON1 pad 164: Net-(CON1-Pad164) -> /D9
- CON1 pad 165: Net-(CON1-Pad165) -> /D24
- CON1 pad 166: Net-(CON1-Pad166) -> GND
- CON1 pad 167: Net-(CON1-Pad167) -> GND
- CON1 pad 168: Net-(CON1-Pad168) -> /D8
- CON1 pad 169: Net-(CON1-Pad169) -> /D16
- CON1 pad 17: Net-(CON1-Pad17) -> /BOSS
- CON1 pad 172: Net-(CON1-Pad172) -> /D0
- CON1 pad 173: Net-(CON1-Pad173) -> /D17
- CON1 pad 174: Net-(CON1-Pad174) -> +5V
- CON1 pad 175: Net-(CON1-Pad175) -> +5V
- CON1 pad 176: Net-(CON1-Pad176) -> /D1
- CON1 pad 177: Net-(CON1-Pad177) -> /D18
- CON1 pad 178: Net-(CON1-Pad178) -> +5V
- CON1 pad 179: Net-(CON1-Pad179) -> +5V
- CON1 pad 18: Net-(CON1-Pad18) -> +5V
- CON1 pad 180: Net-(CON1-Pad180) -> /D2
- CON1 pad 181: Net-(CON1-Pad181) -> /D19
- CON1 pad 182: Net-(CON1-Pad182) -> +5V
- CON1 pad 183: Net-(CON1-Pad183) -> +5V
- CON1 pad 184: Net-(CON1-Pad184) -> /D3
- CON1 pad 185: Net-(CON1-Pad185) -> /D20
- CON1 pad 186: Net-(CON1-Pad186) -> +5V
- CON1 pad 187: Net-(CON1-Pad187) -> +5V
- CON1 pad 188: Net-(CON1-Pad188) -> /D4
- CON1 pad 189: Net-(CON1-Pad189) -> /D21
- CON1 pad 19: Net-(CON1-Pad19) -> +5V
- CON1 pad 190: Net-(CON1-Pad190) -> GND
- CON1 pad 191: Net-(CON1-Pad191) -> GND
- CON1 pad 192: Net-(CON1-Pad192) -> /D5
- CON1 pad 193: Net-(CON1-Pad193) -> /D22
- CON1 pad 194: Net-(CON1-Pad194) -> GND
- CON1 pad 195: Net-(CON1-Pad195) -> GND
- CON1 pad 196: Net-(CON1-Pad196) -> /D6
- CON1 pad 197: Net-(CON1-Pad197) -> /D23
- CON1 pad 198: Net-(CON1-Pad198) -> GND
- CON1 pad 199: Net-(CON1-Pad199) -> GND
- CON1 pad 2: Net-(CON1-Pad2) -> GND
- CON1 pad 20: Net-(CON1-Pad20) -> /FC0
- CON1 pad 200: Net-(CON1-Pad200) -> /D7
- CON1 pad 22: Net-(CON1-Pad22) -> +5V
- CON1 pad 23: Net-(CON1-Pad23) -> +5V
- CON1 pad 24: Net-(CON1-Pad24) -> /FC1
- CON1 pad 25: Net-(CON1-Pad25) -> /BR
- CON1 pad 26: Net-(CON1-Pad26) -> +5V
- CON1 pad 27: Net-(CON1-Pad27) -> +5V
- CON1 pad 29: Net-(CON1-Pad29) -> /BERR
- CON1 pad 3: Net-(CON1-Pad3) -> GND
- CON1 pad 33: Net-(CON1-Pad33) -> /A8
- CON1 pad 35: Net-(CON1-Pad35) -> GND
- CON1 pad 36: Net-(CON1-Pad36) -> /A0
- CON1 pad 37: Net-(CON1-Pad37) -> /A9
- CON1 pad 38: Net-(CON1-Pad38) -> GND
- CON1 pad 39: Net-(CON1-Pad39) -> GND
- CON1 pad 4: Net-(CON1-Pad4) -> /HLT
- CON1 pad 40: Net-(CON1-Pad40) -> /A1
- CON1 pad 41: Net-(CON1-Pad41) -> /A10
- CON1 pad 43: Net-(CON1-Pad43) -> /INT6
- CON1 pad 44: Net-(CON1-Pad44) -> /A2
- CON1 pad 45: Net-(CON1-Pad45) -> /A11
- CON1 pad 47: Net-(CON1-Pad47) -> GND
- CON1 pad 48: Net-(CON1-Pad48) -> /A3
- CON1 pad 49: Net-(CON1-Pad49) -> /A12
- CON1 pad 5: Net-(CON1-Pad5) -> /RW
- CON1 pad 50: Net-(CON1-Pad50) -> GND
- CON1 pad 51: Net-(CON1-Pad51) -> GND
- CON1 pad 52: Net-(CON1-Pad52) -> /A4
- CON1 pad 53: Net-(CON1-Pad53) -> /A13
- CON1 pad 56: Net-(CON1-Pad56) -> /A5
- CON1 pad 57: Net-(CON1-Pad57) -> /A14
- CON1 pad 59: Net-(CON1-Pad59) -> GND
- CON1 pad 6: Net-(CON1-Pad6) -> GND
- CON1 pad 60: Net-(CON1-Pad60) -> /A6
- CON1 pad 61: Net-(CON1-Pad61) -> /A15
- CON1 pad 62: Net-(CON1-Pad62) -> GND
- CON1 pad 63: Net-(CON1-Pad63) -> GND
- CON1 pad 64: Net-(CON1-Pad64) -> /A7
- CON1 pad 65: Net-(CON1-Pad65) -> /A16
- CON1 pad 68: Net-(CON1-Pad68) -> /A24
- CON1 pad 69: Net-(CON1-Pad69) -> /A17
- CON1 pad 7: Net-(CON1-Pad7) -> GND
- CON1 pad 71: Net-(CON1-Pad71) -> GND
- CON1 pad 72: Net-(CON1-Pad72) -> /A25
- CON1 pad 73: Net-(CON1-Pad73) -> /A18
- CON1 pad 74: Net-(CON1-Pad74) -> GND
- CON1 pad 75: Net-(CON1-Pad75) -> GND
- CON1 pad 76: Net-(CON1-Pad76) -> /A26
- CON1 pad 77: Net-(CON1-Pad77) -> /A19
- CON1 pad 8: Net-(CON1-Pad8) -> /BGACK
- CON1 pad 80: Net-(CON1-Pad80) -> /A27
- CON1 pad 81: Net-(CON1-Pad81) -> /A20
- CON1 pad 82: Net-(CON1-Pad82) -> /INT2
- CON1 pad 83: Net-(CON1-Pad83) -> GND
- CON1 pad 84: Net-(CON1-Pad84) -> /A28
- CON1 pad 85: Net-(CON1-Pad85) -> /A21
- CON1 pad 86: Net-(CON1-Pad86) -> GND
- CON1 pad 87: Net-(CON1-Pad87) -> GND
- CON1 pad 88: Net-(CON1-Pad88) -> /A29
- CON1 pad 89: Net-(CON1-Pad89) -> /A22
- CON1 pad 91: Net-(CON1-Pad91) -> /DSACK0
- CON1 pad 92: Net-(CON1-Pad92) -> /A30
- CON1 pad 93: Net-(CON1-Pad93) -> /A23
- CON1 pad 94: Net-(CON1-Pad94) -> +5V
- CON1 pad 95: Net-(CON1-Pad95) -> +5V
- CON1 pad 96: Net-(CON1-Pad96) -> /A31
- CON1 pad 97: Net-(CON1-Pad97) -> /DS
- CON1 pad 98: Net-(CON1-Pad98) -> +5V
- CON1 pad 99: Net-(CON1-Pad99) -> +5V
- CON2 pad 1: Net-(CON2-Pad1) -> /A31
- CON2 pad 10: Net-(CON2-Pad10) -> +5V
- CON2 pad 101: Net-(CON2-Pad101) -> GND
- CON2 pad 102: Net-(CON2-Pad102) -> +5V
- CON2 pad 103: Net-(CON2-Pad103) -> /FC2
- CON2 pad 104: Net-(CON2-Pad104) -> /FC1
- CON2 pad 105: Net-(CON2-Pad105) -> /FC0
- CON2 pad 106: Net-(CON2-Pad106) -> /RMC
- CON2 pad 11: Net-(CON2-Pad11) -> /A23
- CON2 pad 111: Net-(CON2-Pad111) -> /BR
- CON2 pad 112: Net-(CON2-Pad112) -> /BG
- CON2 pad 113: Net-(CON2-Pad113) -> /BGACK
- CON2 pad 114: Net-(CON2-Pad114) -> /BOSS
- CON2 pad 115: Net-(CON2-Pad115) -> /FPUCS
- CON2 pad 118: Net-(CON2-Pad118) -> /RESET
- CON2 pad 119: Net-(CON2-Pad119) -> GND
- CON2 pad 12: Net-(CON2-Pad12) -> /A22
- CON2 pad 120: Net-(CON2-Pad120) -> +5V
- CON2 pad 13: Net-(CON2-Pad13) -> /A21
- CON2 pad 137: Net-(CON2-Pad137) -> /INT2
- CON2 pad 138: Net-(CON2-Pad138) -> /INT6
- CON2 pad 139: Net-(CON2-Pad139) -> GND
- CON2 pad 14: Net-(CON2-Pad14) -> /A20
- CON2 pad 140: Net-(CON2-Pad140) -> +5V
- CON2 pad 146: Net-(CON2-Pad146) -> GND
- CON2 pad 15: Net-(CON2-Pad15) -> /A19
- CON2 pad 16: Net-(CON2-Pad16) -> /A18
- CON2 pad 17: Net-(CON2-Pad17) -> /A17
- CON2 pad 18: Net-(CON2-Pad18) -> /A16
- CON2 pad 19: Net-(CON2-Pad19) -> GND
- CON2 pad 2: Net-(CON2-Pad2) -> /A30
- CON2 pad 20: Net-(CON2-Pad20) -> +5V
- CON2 pad 21: Net-(CON2-Pad21) -> /A15
- CON2 pad 22: Net-(CON2-Pad22) -> /A14
- CON2 pad 23: Net-(CON2-Pad23) -> /A13
- CON2 pad 24: Net-(CON2-Pad24) -> /A12
- CON2 pad 25: Net-(CON2-Pad25) -> /A11
- CON2 pad 26: Net-(CON2-Pad26) -> /A10
- CON2 pad 27: Net-(CON2-Pad27) -> /A9
- CON2 pad 28: Net-(CON2-Pad28) -> /A8
- CON2 pad 29: Net-(CON2-Pad29) -> GND
- CON2 pad 3: Net-(CON2-Pad3) -> /A29
- CON2 pad 30: Net-(CON2-Pad30) -> +5V
- CON2 pad 31: Net-(CON2-Pad31) -> /A7
- CON2 pad 32: Net-(CON2-Pad32) -> /A6
- CON2 pad 33: Net-(CON2-Pad33) -> /A5
- CON2 pad 34: Net-(CON2-Pad34) -> /A4
- CON2 pad 35: Net-(CON2-Pad35) -> /A3
- CON2 pad 36: Net-(CON2-Pad36) -> /A2
- CON2 pad 37: Net-(CON2-Pad37) -> /A1
- CON2 pad 38: Net-(CON2-Pad38) -> /A0
- CON2 pad 39: Net-(CON2-Pad39) -> GND
- CON2 pad 4: Net-(CON2-Pad4) -> /A28
- CON2 pad 40: Net-(CON2-Pad40) -> +5V
- CON2 pad 41: Net-(CON2-Pad41) -> /D31
- CON2 pad 42: Net-(CON2-Pad42) -> /D30
- CON2 pad 43: Net-(CON2-Pad43) -> /D29
- CON2 pad 44: Net-(CON2-Pad44) -> /D28
- CON2 pad 45: Net-(CON2-Pad45) -> /D27
- CON2 pad 46: Net-(CON2-Pad46) -> /D26
- CON2 pad 47: Net-(CON2-Pad47) -> /D25
- CON2 pad 48: Net-(CON2-Pad48) -> /D24
- CON2 pad 49: Net-(CON2-Pad49) -> GND
- CON2 pad 5: Net-(CON2-Pad5) -> /A27
- CON2 pad 50: Net-(CON2-Pad50) -> +5V
- CON2 pad 51: Net-(CON2-Pad51) -> /D23
- CON2 pad 52: Net-(CON2-Pad52) -> /D22
- CON2 pad 53: Net-(CON2-Pad53) -> /D21
- CON2 pad 54: Net-(CON2-Pad54) -> /D20
- CON2 pad 55: Net-(CON2-Pad55) -> /D19
- CON2 pad 56: Net-(CON2-Pad56) -> /D18
- CON2 pad 57: Net-(CON2-Pad57) -> /D17
- CON2 pad 58: Net-(CON2-Pad58) -> /D16
- CON2 pad 59: Net-(CON2-Pad59) -> GND
- CON2 pad 6: Net-(CON2-Pad6) -> /A26
- CON2 pad 60: Net-(CON2-Pad60) -> +5V
- CON2 pad 61: Net-(CON2-Pad61) -> /D15
- CON2 pad 62: Net-(CON2-Pad62) -> /D14
- CON2 pad 63: Net-(CON2-Pad63) -> /D13
- CON2 pad 64: Net-(CON2-Pad64) -> /D12
- CON2 pad 65: Net-(CON2-Pad65) -> /D11
- CON2 pad 66: Net-(CON2-Pad66) -> /D10
- CON2 pad 67: Net-(CON2-Pad67) -> /D9
- CON2 pad 68: Net-(CON2-Pad68) -> /D8
- CON2 pad 69: Net-(CON2-Pad69) -> GND
- CON2 pad 7: Net-(CON2-Pad7) -> /A25
- CON2 pad 70: Net-(CON2-Pad70) -> +5V
- CON2 pad 71: Net-(CON2-Pad71) -> /D7
- CON2 pad 72: Net-(CON2-Pad72) -> /D6
- CON2 pad 73: Net-(CON2-Pad73) -> /D5
- CON2 pad 74: Net-(CON2-Pad74) -> /D4
- CON2 pad 75: Net-(CON2-Pad75) -> /D3
- CON2 pad 76: Net-(CON2-Pad76) -> /D2
- CON2 pad 77: Net-(CON2-Pad77) -> /D1
- CON2 pad 78: Net-(CON2-Pad78) -> /D0
- CON2 pad 79: Net-(CON2-Pad79) -> GND
- CON2 pad 8: Net-(CON2-Pad8) -> /A24
- CON2 pad 80: Net-(CON2-Pad80) -> +5V
- CON2 pad 81: Net-(CON2-Pad81) -> /IPL2
- CON2 pad 82: Net-(CON2-Pad82) -> /IPL1
- CON2 pad 83: Net-(CON2-Pad83) -> /IPL0
- CON2 pad 85: Net-(CON2-Pad85) -> /RST
- CON2 pad 86: Net-(CON2-Pad86) -> /HLT
- CON2 pad 87: Net-(CON2-Pad87) -> /ECS
- CON2 pad 88: Net-(CON2-Pad88) -> /OCS
- CON2 pad 89: Net-(CON2-Pad89) -> /SIZ1
- CON2 pad 9: Net-(CON2-Pad9) -> GND
- CON2 pad 90: Net-(CON2-Pad90) -> /SIZ0
- CON2 pad 91: Net-(CON2-Pad91) -> /AS
- CON2 pad 92: Net-(CON2-Pad92) -> /DS
- CON2 pad 93: Net-(CON2-Pad93) -> /RW
- CON2 pad 94: Net-(CON2-Pad94) -> /BERR
- CON2 pad 96: Net-(CON2-Pad96) -> /AVEC
- CON2 pad 97: Net-(CON2-Pad97) -> /DSACK1
- CON2 pad 98: Net-(CON2-Pad98) -> /DSACK0
- CON2 pad 99: Net-(CON2-Pad99) -> /CPUCLK
Routing:
- added copper zone on In1.Cu_(5V), net +5V
- added copper zone on In2.Cu_(GND), net GND
Other:
- copper layers 2 -> 4
- board text added: "A3000/4000 to A1200 Pistorm32 Adapter"
- board text removed: "A3000/4000 to A1200 CPU Adapter"
