File: A1200-adapter/A1200-adapter.sch (KiCad schematic (older format))
At the start: 2 parts, among them CON1 A3000_A4000_LOCAL_BUS_SLOT, CON2 A1200-EXP

Commit message: Add files via upload
Connections:
- net DSACK1: now reaches CON1.1 (_DSACK1)
- net DSACK1: now also CON2.97 (DSACK_1)
- net GND: now reaches CON1.10 (GND)
- net GND: now also CON1.11 (GND), CON1.115 (GND), CON1.118 (GND), CON1.119 (GND), CON1.127 (GND), CON1.130 (GND), CON1.131 (GND), CON1.138 (GND), CON1.139 (GND), CON1.142 (GND), CON1.143 (GND), CON1.151 (GND), CON1.154 (GND), CON1.155 (GND), CON1.163 (GND), CON1.166 (GND), CON1.167 (GND), CON1.190 (GND), CON1.191 (GND), CON1.194 (GND), CON1.195 (GND), CON1.198 (GND), CON1.199 (GND), CON1.2 (GND), CON1.3 (GND), CON1.35 (GND), CON1.38 (GND), CON1.39 (GND), CON1.47 (GND), CON1.50 (GND), CON1.51 (GND), CON1.59 (GND), CON1.6 (GND), CON1.62 (GND), CON1.63 (GND), CON1.7 (GND), CON1.71 (GND), CON1.74 (GND), CON1.75 (GND), CON1.83 (GND), CON1.86 (GND), CON1.87 (GND), CON2.101 (GND), CON2.119 (GND), CON2.139 (GND), CON2.146 (AUDIO_GND), CON2.19 (GND), CON2.29 (GND), CON2.39 (GND), CON2.49 (GND), CON2.59 (GND), CON2.69 (GND), CON2.79 (GND), CON2.9 (GND)
- net ECS: now reaches CON1.100 (_ECS)
- net ECS: now also CON2.87 (ECS)
- net +5V: now reaches CON1.102 (+5V)
- net +5V: now also CON1.103 (+5V), CON1.106 (+5V), CON1.107 (+5V), CON1.14 (+5V), CON1.15 (+5V), CON1.174 (+5V), CON1.175 (+5V), CON1.178 (+5V), CON1.179 (+5V), CON1.18 (+5V), CON1.182 (+5V), CON1.183 (+5V), CON1.186 (+5V), CON1.187 (+5V), CON1.19 (+5V), CON1.22 (+5V), CON1.23 (+5V), CON1.26 (+5V), CON1.27 (+5V), CON1.94 (+5V), CON1.95 (+5V), CON1.98 (+5V), CON1.99 (+5V), CON2.10 (VCC), CON2.102 (VCC), CON2.120 (VCC), CON2.140 (VCC), CON2.20 (VCC), CON2.30 (VCC), CON2.40 (VCC), CON2.50 (VCC), CON2.60 (VCC), CON2.70 (VCC), CON2.80 (VCC)
- net BG: now reaches CON1.105 (_BG)
- net BG: now also CON2.112 (BG)
- net RMC: now reaches CON1.108 (_RMC)
- net RMC: now also CON2.106 (RMC)
- net RST: now reaches CON1.109 (_CPURST)
- net RST: now also CON2.85 (RST)
- net RESET: now reaches CON1.117 (_RESET)
- net RESET: now also CON2.118 (RESET)
- net AVEC: now reaches CON1.12 (_AVEC)
- net AVEC: now also CON2.96 (AVEC)
- net IPL0: now reaches CON1.120 (IPL0)
- net IPL0: now also CON2.83 (IPL0)
- net SIZ0: now reaches CON1.121 (SIZ0)
- net SIZ0: now also CON2.90 (SIZE_0)
- net IPL1: now reaches CON1.124 (IPL1)
- net IPL1: now also CON2.82 (IPL1)
- net FC2: now reaches CON1.125 (FC2)
- net FC2: now also CON2.103 (FC2)
- net IPL2: now reaches CON1.128 (IPL2)
- net IPL2: now also CON2.81 (IPL2)
- net SIZ1: now reaches CON1.129 (SIZ1)
- net SIZ1: now also CON2.89 (SIZE_1)
- net AS: now reaches CON1.133 (_AS)
- net AS: now also CON2.91 (AS)
- net FPUCS: now reaches CON1.134 (_FPUCS)
- net FPUCS: now also CON2.115 (FPU_CS)
- net CPUCLK: now reaches CON1.135 (CPUCLK_EXP)
- net CPUCLK: now also CON2.99 (CPUCLK_A)
- net OCS: now reaches CON1.136 (_OCS)
- net OCS: now also CON2.88 (OCS)
- net D31: now reaches CON1.137 (D31)
- net D31: now also CON2.41 (D31)
- net D15: now reaches CON1.140 (D15)
- net D15: now also CON2.61 (D15)
- net D30: now reaches CON1.141 (D30)
- net D30: now also CON2.42 (D30)
- net D14: now reaches CON1.144 (D14)
- net D14: now also CON2.62 (D14)
- net D29: now reaches CON1.145 (D29)
- net D29: now also CON2.43 (D29)
- net D13: now reaches CON1.148 (D13)
- net D13: now also CON2.63 (D13)
- net D28: now reaches CON1.149 (D28)
- net D28: now also CON2.44 (D28)
- net D12: now reaches CON1.152 (D12)
- net D12: now also CON2.64 (D12)
- net D27: now reaches CON1.153 (D27)
- net D27: now also CON2.45 (D27)
- net D11: now reaches CON1.156 (D11)
- net D11: now also CON2.65 (D11)
- net D26: now reaches CON1.157 (D26)
- net D26: now also CON2.46 (D26)
- net D10: now reaches CON1.160 (D10)
- net D10: now also CON2.66 (D10)
- net D25: now reaches CON1.161 (D25)
- net D25: now also CON2.47 (D25)
- net D9: now reaches CON1.164 (D9)
- net D9: now also CON2.67 (D9)
- net D24: now reaches CON1.165 (D24)
- net D24: now also CON2.48 (D24)
- net D8: now reaches CON1.168 (D8)
- net D8: now also CON2.68 (D8)
- net D16: now reaches CON1.169 (D16)
- net D16: now also CON2.58 (D16)
- net BOSS: now reaches CON1.17 (_BOSS)
- net BOSS: now also CON2.114 (BOSS)
- net D0: now reaches CON1.172 (D0)
- net D0: now also CON2.78 (D0)
- net D17: now reaches CON1.173 (D17)
- net D17: now also CON2.57 (D17)
- net D1: now reaches CON1.176 (D1)
- net D1: now also CON2.77 (D1)
- net D18: now reaches CON1.177 (D18)
- net D18: now also CON2.56 (D18)
- net D2: now reaches CON1.180 (D2)
- net D2: now also CON2.76 (D2)
- net D19: now reaches CON1.181 (D19)
- net D19: now also CON2.55 (D19)
- net D3: now reaches CON1.184 (D3)
- net D3: now also CON2.75 (D3)
- net D20: now reaches CON1.185 (D20)
- net D20: now also CON2.54 (D20)
- net D4: now reaches CON1.188 (D4)
- net D4: now also CON2.74 (D4)
- net D21: now reaches CON1.189 (D21)
- net D21: now also CON2.53 (D21)
- net D5: now reaches CON1.192 (D5)
- net D5: now also CON2.73 (D5)
- net D22: now reaches CON1.193 (D22)
- net D22: now also CON2.52 (D22)
- net D6: now reaches CON1.196 (D6)
- net D6: now also CON2.72 (D6)
- net D23: now reaches CON1.197 (D23)
- net D23: now also CON2.51 (D23)
- net FC0: now reaches CON1.20 (FC0)
- net FC0: now also CON2.105 (FC0)
- net D7: now reaches CON1.200 (D7)
- net D7: now also CON2.71 (D7)
- net FC1: now reaches CON1.24 (FC1)
- net FC1: now also CON2.104 (FC1)
- net BR: now reaches CON1.25 (_BR)
- net BR: now also CON2.111 (BR)
- net BERR: now reaches CON1.29 (_BERR)
- net BERR: now also CON2.94 (BEER)
- net A8: now reaches CON1.33 (A8)
- net A8: now also CON2.28 (A8)
- net A0: now reaches CON1.36 (A0)
- net A0: now also CON2.38 (A0)
- net A9: now reaches CON1.37 (A9)
- net A9: now also CON2.27 (A9)
- net HLT: now reaches CON1.4 (_HLT)
- net HLT: now also CON2.86 (HLT)
- net A1: now reaches CON1.40 (A1)
- net A1: now also CON2.37 (A1)
- net A10: now reaches CON1.41 (A10)
- net A10: now also CON2.26 (A10)
- net INT6: now reaches CON1.43 (_INT6)
- net INT6: now also CON2.138 (INT6)
- net A2: now reaches CON1.44 (A2)
- net A2: now also CON2.36 (A2)
- net A11: now reaches CON1.45 (A11)
- net A11: now also CON2.25 (A11)
- net A3: now reaches CON1.48 (A3)
- net A3: now also CON2.35 (A3)
- net A12: now reaches CON1.49 (A12)
- net A12: now also CON2.24 (A12)
- net RW: now reaches CON1.5 (R_W)
- net RW: now also CON2.93 (R_W)
- net A4: now reaches CON1.52 (A4)
- net A4: now also CON2.34 (A4)
- net A13: now reaches CON1.53 (A13)
- net A13: now also CON2.23 (A13)
- net A5: now reaches CON1.56 (A5)
- net A5: now also CON2.33 (A5)
- net A14: now reaches CON1.57 (A14)
- net A14: now also CON2.22 (A14)
- net A6: now reaches CON1.60 (A6)
- net A6: now also CON2.32 (A6)
- net A15: now reaches CON1.61 (A15)
- net A15: now also CON2.21 (A15)
- net A7: now reaches CON1.64 (A7)
- net A7: now also CON2.31 (A7)
- net A16: now reaches CON1.65 (A16)
- net A16: now also CON2.18 (A16)
- net A24: now reaches CON1.68 (MA24)
- net A24: now also CON2.8 (A24)
- net A17: now reaches CON1.69 (A17)
- net A17: now also CON2.17 (A17)
- net A25: now reaches CON1.72 (MA25)
- net A25: now also CON2.7 (A25)
- net A18: now reaches CON1.73 (A18)
- net A18: now also CON2.16 (A18)
- net A26: now reaches CON1.76 (MA26)
- net A26: now also CON2.6 (A26)
- net A19: now reaches CON1.77 (A19)
- net A19: now also CON2.15 (A19)
- net BGACK: now reaches CON1.8 (_BGACK)
- net BGACK: now also CON2.113 (BGACK)
- net A27: now reaches CON1.80 (A27)
- net A27: now also CON2.5 (A27)
- net A20: now reaches CON1.81 (A20)
- net A20: now also CON2.14 (A20)
- net INT2: now reaches CON1.82 (INT2)
- net INT2: now also CON2.137 (INT2)
- net A28: now reaches CON1.84 (A28)
- net A28: now also CON2.4 (A28)
- net A21: now reaches CON1.85 (A21)
- net A21: now also CON2.13 (A21)
- net A29: now reaches CON1.88 (A29)
- net A29: now also CON2.3 (A29)
- net A22: now reaches CON1.89 (A22)
- net A22: now also CON2.12 (A22)
- net DSACK0: now reaches CON1.91 (_DSACK0)
- net DSACK0: now also CON2.98 (DSACK_0)
- net A30: now reaches CON1.92 (A30)
- net A30: now also CON2.2 (A30)
- net A23: now reaches CON1.93 (A23)
- net A23: now also CON2.11 (A23)
- net A31: now reaches CON1.96 (A31)
- net A31: now also CON2.1 (A31)
- net DS: now reaches CON1.97 (_DS)
- net DS: now also CON2.92 (DS)
- no-connect marks 0 -> 74
Other:
- note added: "*No-connects here go nowhere on Pistorm32 per its schematic."
- moved on the sheet: CON1
